File: 0102-USB-SWITCH.kicad_sch (KiCad schematic)
At the start: 11 parts, among them J1 UPSTREAM, J2 DOWNSTREAM, SW1 EN

Commit message: Rework PCB for kibuzzard silk and laying USB-A slot
Parts:
- J2: footprint JLC-SMT:CKMTW_USBAS04P -> JLC-SMT:MOLEX_48258-0001
Changed lines of the file:
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@@
     (property "Reference" "J2" (id 0) (at 184.3278 46.5582 0))
     (property "Value" "DOWNSTREAM" (id 1) (at 184.3278 48.8696 0))
-    (property "Footprint" "JLC-SMT:CKMTW_USBAS04P" (id 2) (at 186.69 59.69 0)
+    (property "Footprint" "JLC-SMT:MOLEX_48258-0001" (id 2) (at 186.69 59.69 0)
       (effects (font (size 1.27 1.27)) hide)
     )
@@
     )
     (path "/00000000-0000-0000-0000-0000630bb6fc"
-      (reference "J2") (unit 1) (value "DOWNSTREAM") (footprint "JLC-SMT:CKMTW_USBAS04P")
+      (reference "J2") (unit 1) (value "DOWNSTREAM") (footprint "JLC-SMT:MOLEX_48258-0001")
     )
     (path "/00000000-0000-0000-0000-00006306f344"

Commit message: Output docs
Parts:
- J2: Manufacturer Ckmtw -> MOLEX; PartNumber C386737 -> C505080; Supplier JLC-EXT -> LCSC
Changed lines of the file:
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@@
   (title_block
     (title "#0102 USB SWITCH")
+    (date "2022-09-13")
     (rev "V1.1")
     (company "TileParts")
@@
       (effects (font (size 1.27 1.27)) hide)
     )
-    (property "Manufacturer" "Ckmtw" (id 4) (at 182.88 58.42 0)
-      (effects (font (size 1.27 1.27)) hide)
-    )
-    (property "PartNumber" "C386737" (id 5) (at 182.88 58.42 0)
-      (effects (font (size 1.27 1.27)) hide)
-    )
-    (property "Supplier" "JLC-EXT" (id 6) (at 182.88 58.42 0)
-      (effects (font (size 1.27 1.27)) hide)
-    )
+    (property "Manufacturer" "MOLEX" (id 4) (at 182.88 58.42 0)
+      (effects (font (size 1.27 1.27)) hide)
+    )
+    (property "PartNumber" "C505080" (id 5) (at 182.88 58.42 0)
+      (effects (font (size 1.27 1.27)) hide)
+    )
+    (property "Supplier" "LCSC" (id 6) (at 182.88 58.42 0)
+      (effects (font (size 1.27 1.27)) hide)
+    )

Commit message: Rework with new design
Parts:
- removed H1, H2, H3: MountingHole, MountingHole:MountingHole_2.2mm_M2, symbol Mechanical:MountingHole
- J1: footprint JLC-SMT:KINGHELM_KH-TYPE-C-L10-14P -> JLC-SMT:HRO_TYPE-C-31-M-12; Manufacturer kinghelm -> HRO; PartNumber C2761226 -> (none)
Connections:
- net GND: now also J1.S1 (SHIELD), J2.5 (Shield)
- no-connect marks 8 -> 6
Changed lines of the file:
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@@
   (title_block
     (title "#0102 USB SWITCH")
-    (date "2022-09-13")
-    (rev "V1.1")
+    (date "2022-09-23")
+    (rev "V1.2")
     (company "TileParts")
   )
@@
   )
   (junction (at 76.2 68.58) (diameter 0) (color 0 0 0 0)
+  )
+  (junction (at 182.88 68.58) (diameter 0) (color 0 0 0 0)
   )
   (junction (at 124.46 55.88) (diameter 0) (color 0 0 0 0)
@@
   (no_connect (at 76.2 81.28))
   (no_connect (at 111.76 60.96))
-  (no_connect (at 53.34 91.44))
-  (no_connect (at 180.34 68.58))
   (wire (pts (xy 195.58 60.96) (xy 190.5 60.96))
     (stroke (width 0) (type default) (color 0 0 0 0))
@@
   )
   (wire (pts (xy 81.28 68.58) (xy 76.2 68.58))
+    (stroke (width 0) (type default) (color 0 0 0 0))
+  )
+  (wire (pts (xy 180.34 68.58) (xy 182.88 68.58))
     (stroke (width 0) (type default) (color 0 0 0 0))
   )
@@
     (property "Reference" "J1" (id 0) (at 63.6778 46.5582 0))
     (property "Value" "UPSTREAM" (id 1) (at 63.6778 48.8696 0))
-    (property "Footprint" "JLC-SMT:KINGHELM_KH-TYPE-C-L10-14P" (id 2) (at 64.77 68.58 0)
+    (property "Footprint" "JLC-SMT:HRO_TYPE-C-31-M-12" (id 2) (at 64.77 68.58 0)
       (effects (font (size 1.27 1.27)) hide)
     )
@@
       (effects (font (size 1.27 1.27)) hide)
     )
-    (property "Manufacturer" "kinghelm" (id 4) (at 60.96 68.58 0)
-      (effects (font (size 1.27 1.27)) hide)
-    )
-    (property "PartNumber" "C2761226" (id 5) (at 60.96 68.58 0)
+    (property "Manufacturer" "HRO" (id 4) (at 60.96 68.58 0)
+      (effects (font (size 1.27 1.27)) hide)
+    )
+    (property "PartNumber" "" (id 5) (at 60.96 68.58 0)
       (effects (font (size 1.27 1.27)) hide)
     )
@@
     (pin "1")
   )
-  (symbol (lib_id "Mechanical:MountingHole") (at 114.3 114.3 0) (unit 1)
-    (in_bom yes) (on_board yes)
-    (property "Reference" "H1" (id 0) (at 116.84 113.1316 0)
-      (effects (font (size 1.27 1.27)) (justify left))
-    )
-    (property "Value" "MountingHole" (id 1) (at 116.84 115.443 0)
-      (effects (font (size 1.27 1.27)) (justify left))
-    )
-    (property "Footprint" "MountingHole:MountingHole_2.2mm_M2" (id 2) (at 114.3 114.3 0)
-      (effects (font (size 1.27 1.27)) hide)
-    )
-    (property "Datasheet" "~" (id 3) (at 114.3 114.3 0)
-      (effects (font (size 1.27 1.27)) hide)
-    )
-    (property "Manufacturer" "~" (id 4) (at 114.3 114.3 0)
-      (effects (font (size 1.27 1.27)) hide)
-    )
-    (property "PartNumber" "~" (id 5) (at 114.3 114.3 0)
-      (effects (font (size 1.27 1.27)) hide)
-    )
-    (property "Supplier" "~" (id 6) (at 114.3 114.3 0)
-      (effects (font (size 1.27 1.27)) hide)
-    )
-  )
-  (symbol (lib_id "Mechanical:MountingHole") (at 114.3 127 0) (unit 1)
-    (in_bom yes) (on_board yes)
-    (property "Reference" "H2" (id 0) (at 116.84 125.8316 0)
-      (effects (font (size 1.27 1.27)) (justify left))
-    )
-    (property "Value" "MountingHole" (id 1) (at 116.84 128.143 0)
-      (effects (font (size 1.27 1.27)) (justify left))
-    )
-    (property "Footprint" "MountingHole:MountingHole_2.2mm_M2" (id 2) (at 114.3 127 0)
-      (effects (font (size 1.27 1.27)) hide)
-    )
-    (property "Datasheet" "~" (id 3) (at 114.3 127 0)
-      (effects (font (size 1.27 1.27)) hide)
-    )
-    (property "Manufacturer" "~" (id 4) (at 114.3 127 0)
-      (effects (font (size 1.27 1.27)) hide)
-    )
-    (property "PartNumber" "~" (id 5) (at 114.3 127 0)
-      (effects (font (size 1.27 1.27)) hide)
-    )
-    (property "Supplier" "~" (id 6) (at 114.3 127 0)
-      (effects (font (size 1.27 1.27)) hide)
-    )
-  )
-  (symbol (lib_id "Mechanical:MountingHole") (at 114.3 139.7 0) (unit 1)
-    (in_bom yes) (on_board yes)
-    (property "Reference" "H3" (id 0) (at 116.84 138.5316 0)
-      (effects (font (size 1.27 1.27)) (justify left))
-    )
-    (property "Value" "MountingHole" (id 1) (at 116.84 140.843 0)
-      (effects (font (size 1.27 1.27)) (justify left))
-    )
-    (property "Footprint" "MountingHole:MountingHole_2.2mm_M2" (id 2) (at 114.3 139.7 0)
-      (effects (font (size 1.27 1.27)) hide)
-    )
-    (property "Datasheet" "~" (id 3) (at 114.3 139.7 0)
-      (effects (font (size 1.27 1.27)) hide)
-    )
-    (property "Manufacturer" "~" (id 4) (at 114.3 139.7 0)
-      (effects (font (size 1.27 1.27)) hide)
-    )
-    (property "PartNumber" "~" (id 5) (at 114.3 139.7 0)
-      (effects (font (size 1.27 1.27)) hide)
-    )
-    (property "Supplier" "~" (id 6) (at 114.3 139.7 0)
-      (effects (font (size 1.27 1.27)) hide)
-    )
-  )
   (symbol (lib_id "Device:R_US") (at 85.09 60.96 270) (unit 1)
     (in_bom yes) (on_board yes)
@@
     (pin "5")
   )
+  (symbol (lib_id "power:GND") (at 53.34 91.44 0) (unit 1)
+    (in_bom yes) (on_board yes)
+    (property "Reference" "#PWR0101" (id 0) (at 53.34 97.79 0)
+      (effects (font (size 1.27 1.27)) hide)
+    )
+    (property "Value" "GND" (id 1) (at 53.467 95.8342 0)
+      (effects (font (size 1.27 1.27)) hide)
+    )
+    (property "Footprint" "" (id 2) (at 53.34 91.44 0)
+      (effects (font (size 1.27 1.27)) hide)
+    )
+    (property "Datasheet" "" (id 3) (at 53.34 91.44 0)
+      (effects (font (size 1.27 1.27)) hide)
+    )
+    (pin "1")
+  )
   (sheet_instances
     (path "/" (page "1"))
@@
       (reference "#PWR05") (unit 1) (value "GND") (footprint "")
     )
+    (path "/66efefc7-4e2b-4327-ac28-0db3f480ad77"
+      (reference "#PWR0101") (unit 1) (value "GND") (footprint "")
+    )
     (path "/00000000-0000-0000-0000-000063072038"
       (reference "D1") (unit 1) (value "POWER") (footprint "LED_SMD:LED_0603_1608Metric")
     )
-    (path "/00000000-0000-0000-0000-000063082217"
-      (reference "H1") (unit 1) (value "MountingHole") (footprint "MountingHole:MountingHole_2.2mm_M2")
-    )
-    (path "/00000000-0000-0000-0000-0000630827a3"
-      (reference "H2") (unit 1) (value "MountingHole") (footprint "MountingHole:MountingHole_2.2mm_M2")
-    )
-    (path "/00000000-0000-0000-0000-000063089fe0"
-      (reference "H3") (unit 1) (value "MountingHole") (footprint "MountingHole:MountingHole_2.2mm_M2")
-    )
     (path "/00000000-0000-0000-0000-00006305bc90"
-      (reference "J1") (unit 1) (value "UPSTREAM") (footprint "JLC-SMT:KINGHELM_KH-TYPE-C-L10-14P")
+      (reference "J1") (unit 1) (value "UPSTREAM") (footprint "JLC-SMT:HRO_TYPE-C-31-M-12")
     )
     (path "/00000000-0000-0000-0000-0000630bb6fc"

Commit message: Output MF docs V1.2
Parts:
- J1: PartNumber (none) -> C165948
Changed lines of the file:
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@@
       (effects (font (size 1.27 1.27)) hide)
     )
-    (property "PartNumber" "" (id 5) (at 60.96 68.58 0)
+    (property "PartNumber" "C165948" (id 5) (at 60.96 68.58 0)
       (effects (font (size 1.27 1.27)) hide)
     )
